Commit message: ROS2 Galactic and parameter changes

File: config/robot.urdf.xacro (robot description, xacro)
@@ -33,3 +33,9 @@
     <origin xyz="0 0 0" rpy="0 0 0" />
   </joint>
+  <link name="map"> </link>
+  <joint name="map_joint" type="fixed">
+    <parent link="chassis_link" />
+    <child link="map" />
+    <origin xyz="0 0 0" rpy="0 0 0" />
+  </joint>
 </robot>
